File: icm7212m-display.kicad_pcb (KiCad board)
At the start: 2 copper layers, 70 x 60 mm, 12 parts, among them J1 Conn_01x10_Socket, U1 ICM7212M, U2 SM410561N, U3 SM410561N, U4 SM410561N, U5 SM410561N

Commit message: additional refinement
Parts:
- moved C1 0.78 mm to (105.7, 76.8)
- moved J1 0.78 mm to (121.2, 56.5)
- moved RV1 0.78 mm to (106.7, 66.0)
- moved U1 0.78 mm to (111.0, 76.7)
- moved U2 0.78 mm to (110.5, 102.1)
- moved U3 0.78 mm to (123.5, 102.1)
- moved U4 0.78 mm to (136.5, 102.1)
- moved U5 0.78 mm to (149.5, 102.1)
Routing:
- net VCC: track 137.1 -> 154.2 mm
- net Net-(J1-Pin_8): track 0.09 -> 5.05 mm
- net Net-(J1-Pin_9): track 0.09 -> 5.05 mm
- net Net-(J1-Pin_7): track 0.09 -> 5.05 mm
- net Net-(J1-Pin_6): track 0.09 -> 5.05 mm
- net Net-(J1-Pin_5): track 0.09 -> 5.05 mm
- net Net-(J1-Pin_4): track 0.09 -> 5.05 mm
- net Net-(J1-Pin_3): track 0.09 -> 5.05 mm
- net Net-(J1-Pin_10): track 0.09 -> 5.05 mm
Other:
- outline, holes or cut-outs redrawn
- board text added: "ICM7212M LED Display Module"
- board text removed: "ICM7212M"
