File: icm7212m-display.kicad_sch (KiCad schematic)
At the start: 12 parts, among them J1 Conn_01x10_Socket, U1 ICM7212M, U2 SM410561N, U3 SM410561N, U4 SM410561N, U5 SM410561N

Commit message: add PDF for the schematic
Other:
- title: (none) -> ICM7212M Display Module
Changed lines of the file:
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@@
 	(generator_version "9.0")
 	(paper "A4")
+	(title_block
+		(title "ICM7212M Display Module")
+		(date "2025-06-19")
+		(rev "1")
+	)
 	(junction
 		(at 208.28 120.65)
